File: kicad/DisplayModule_PONSv5.kicad_sch (KiCad schematic)
At the start: 38 parts, among them J1 Ext. Speaker, J3 541324062, J4 Micro_SD_Card_Det2, J5 Conn_01x14_Pin, Q2 DMG3415U, SW1 SW0_BOARD, SW3 BAT_TFT_SW, U1 Pico, U2 MCP73831-2-OT, U3 LC86GPAMD, U4 PAM8304ASR

Commit message: Kicad
Kicad for hardware v5
Parts:
- removed J3: 541324062, Connector_Molex:CON_541324062_MOL, symbol Connector:541324062
- removed J5: Conn_01x14_Pin, Connector_PinHeader_2.54mm:PinHeader_1x14_P2.54mm_Vertical, symbol Connector:Conn_01x14_Pin
- removed LS1: UM1515IA, Buzzer_Beeper:UM1515IA085008, symbol Device:Speaker
- removed R1: 470, Resistor_SMD:R_0603_1608Metric_Pad0.98x0.95mm_HandSolder, symbol Device:R
- removed RSTSW1: RSTSW_BOARD, Button_Switch_SMD:TVAF06-A020B-R, symbol Switch:SW_Push
- removed U3: LC86GPAMD, RF_GPS:L86_QWS, symbol RF_GPS:L86-M33
- removed U4: PAM8304ASR, Package_SO:MSOP-8-1EP_3x3mm_P0.65mm_EP1.5x1.8mm, symbol Amplifier_Audio:PAM8304ASR
- added C10: 0.1u, Capacitor_SMD:C_0603_1608Metric_Pad1.08x0.95mm_HandSolder, symbol Device:C
- added C11, C12: 220p, Capacitor_SMD:C_0603_1608Metric_Pad1.08x0.95mm_HandSolder, symbol Device:C
- added C13, C15: (220u), Capacitor_SMD:C_1210_3225Metric_Pad1.33x2.70mm_HandSolder, symbol Device:C
- added C14: 4.7u, Capacitor_SMD:C_0603_1608Metric_Pad1.08x0.95mm_HandSolder, symbol Device:C
- added FB1, FB2: 120, Inductor_SMD:L_1206_3216Metric_Pad1.22x1.90mm_HandSolder, symbol Device:FerriteBead_Small
- added J2: 541324062, Connector_Molex:CON_541324062_MOL, symbol Connector:541324062_NHD
- added J5: Conn_01x03_Pin, Connector_PinHeader_2.54mm:PinHeader_1x03_P2.54mm_Vertical, symbol Connector:Conn_01x03_Pin
- added J6: Conn_01x05_Pin, Connector_PinHeader_2.54mm:PinHeader_1x05_P2.54mm_Vertical, symbol Connector:Conn_01x05_Pin
- added R10: 1.2k, Resistor_SMD:R_0603_1608Metric_Pad0.98x0.95mm_HandSolder, symbol Device:R
- added R11, R12, R13, R14, R15, R16: 47, Resistor_SMD:R_0603_1608Metric_Pad0.98x0.95mm_HandSolder, symbol Device:R
- added R17, R18, R19, R20, R21, R22: 4.7k, Resistor_SMD:R_0603_1608Metric_Pad0.98x0.95mm_HandSolder, symbol Device:R
- added RV1: 100k, Potentiometer_SMD:Potentiometer_PVZ3A, symbol Device:R_Potentiometer
- added U3: LC86GPAMD, RF_GPS:L86_QWS, symbol RF_GPS:LC86GPAMD
- added U4: PAM8302AAD, Package_SO:SO-8_3.9x4.9mm_P1.27mm, symbol Amplifier_Audio:PAM8302AAD
- C2, C4: value 100n -> 0.1u
- C5, C6: value 100n -> 1u
- C8: value 1u -> (1500u); footprint Capacitor_SMD:C_0603_1608Metric_Pad1.08x0.95mm_HandSolder -> Capacitor_SMD:CP_Elec_10x10.5
- C9: value (47u) -> 47u
- J1: footprint Connector_JST:JST_XA_B02B-XASK-1_1x02_P2.50mm_Vertical -> Connector_JST:JST_XH_S2B-XH-A-1_1x02_P2.50mm_Horizontal
- R8, R9: value 1M -> 100
Connections:
- net DB2 is gone; now on net SD_DETA: U1.11 (GPIO8)
- net SW_RUN is gone; now on net +3.3V: U1.30 (RUN)
- net +3.3V: now also C13.1, C14.1, C15.1, J2.10 (31), J2.28 (13), J2.33 (8), J2.34 (7), J6.1 (Pin_1), R17.2, R18.2, R19.2, R20.2, R21.2, R22.2, U3.4 (VCC), U4.6 (VDD)
- net DB10: now also J2.17 (24)
- net DB11: now also J2.16 (25)
- net DB12: now also J2.15 (26)
- net DB13: now also J2.14 (27)
- net DB14: now also J2.13 (28)
- net DB15: now also J2.12 (29)
- net DB8: now also J2.19 (22)
- net DB9: now also J2.18 (23)
- net GND: now also J4.11 (SHIELD), J4.9 (DET_B), U1.42 (GND), C10.1, C11.2, C12.2, C13.2, C14.2, C15.2, J2.2 (39), J2.31 (10), J2.4 (37), J2.40 (1), J2.5 (36), J2.6 (35), J2.7 (34), J2.8 (33), J5.2 (Pin_2), J6.2 (Pin_2), RV1.3, U3.12 (GND), U3.3 (GND), U4.7 (GND); no longer J4.2 (DAT3/CD)
- net TFT_DC: now also U1.34 (GPIO28_ADC2), J2.30 (11); no longer U1.32 (GPIO27_ADC1)
- net TFT_RESET: now also J2.11 (30)
- net TFT_WR: now also U1.32 (GPIO27_ADC1), J2.29 (12); no longer U1.34 (GPIO28_ADC2)
- net UART1_RX: now also U3.2 (TXD1)
- net UART1_TX: now also U3.1 (RXD1)
- net at R8.2: now also U4.4 (IN-)
- net at U1.41 (SWCLK): now also J5.1 (Pin_1)
- net at U1.43 (SWDIO): now also J5.3 (Pin_3)
- net at BT1.1 (+), C1.1, C2.1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: now also U3.5 (V_BCKP)
- net at J1.1 (Pin_1): now also C11.1, FB1.2
- net at J1.2 (Pin_2): now also C12.1, FB2.2
- net at R3.2, R4.2: now also J2.3 (38)
- net at R9.2: now also U4.3 (IN+)
- net at J4.1 (DAT2): now also R11.2, R17.1
- net SD_DETA: now reaches J4.10 (DET_A)
- net at J4.8 (DAT1): now also R16.2, R22.1
- net ADC_VREF: no longer names the net of U1.35 (ADC_VREF)
- net DB0 renamed SD_DAT2
- net SD_DAT2: now also R11.1
- net DB1 renamed SD_DAT3
- net SD_DAT3: now also R12.1
- net DB3 renamed PWM_AUDIO
- net PWM_AUDIO: now also R10.2
- net DB4 renamed AMP_SD
- net AMP_SD: now also U4.1 (~{SD})
- net DB5 renamed GPIO11
- net GPIO11: now also J6.3 (Pin_3)
- net DB6 renamed GPIO12
- net GPIO12: now also J6.4 (Pin_4)
- net DB7 renamed GPIO13
- net GPIO13: now also J6.5 (Pin_5)
- net GPIO5: no longer names the net of C6.1
- net GPIO5: now also RV1.2; no longer U1.7 (GPIO5)
- net SPI0_MISO_GPIO4: no longer names the net of J4.7 (DAT0)
- net SPI0_MISO_GPIO4: now also R15.2, R21.1; no longer U1.6 (GPIO4)
- net SPI0_MOSI_GPIO3: no longer names the net of J4.3 (CMD)
- net SPI0_MOSI_GPIO3: now also R13.2, R19.1; no longer U1.5 (GPIO3)
- net SPI0_SCL_GPIO2: no longer names the net of J4.5 (CLK)
- net SPI0_SCL_GPIO2: now also R14.2, R20.1; no longer U1.4 (GPIO2)
- new net: J4.2 (DAT3/CD), R12.2, R18.1
- new net: C10.2, R10.1, RV1.1
- new net: FB2.1, U4.5 (OUT+)
- new net: FB1.1, U4.8 (OUT-)
- new net SD_CLK: R14.1, U1.4 (GPIO2)
- new net SD_CMD: R13.1, U1.5 (GPIO3)
- new net SD_DAT0: R15.1, U1.6 (GPIO4)
- new net SD_DAT1: R16.1, U1.7 (GPIO5)
- no-connect marks 0 -> 7
Other:
- note added: "(0.1uF+1kΩ Acceptable)"
- note added: "2.2k to limit current"
- note added: "BLM31PG121SN1L"
- note added: "GNSS"
- note added: "Optional SDIO"
- note removed: "Optional GPS"
- note removed: "Optional SD"
- moved on the sheet: BT1, C1, C2, C3, C4, C5, C6, C7, C9, D1, D2, J1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
