File: kicad/mainboard/DisplayModule_PONSv7.kicad_pcb (KiCad board)
At the start: 4 copper layers, 55.4 x 77.6 mm, 135 parts, among them J1 Ext. Speaker, J2 54132-4062, J3 2005280040, J4 Micro_SD_Card_Det2, J5 Conn_01x03_Shielded, J6 USB_B_Micro, Q1 AO3401A, SW1 PTS645VK392LFS, SW2 SW_TS-1088, SW3 SW_TS-1088, U1 PAM8302AADCR, U10 BNO085, U12 E220-900T22S(JP), U2 W25Q128JVS, U3 RP2350_80QFN, U4 MCP73831-2-OT, U5 TPS63031DSK, U6 MAINSW_CUS-12TB, U7 TFTSW_CUS-12TB, U8 MS5611-01BA, Y1 X322512MSB4SI, Y2 32.768k

Commit message: 0.961 KiCad更新 wav更新
wav雑音除去
kicad更新（スイッチ背面、DocへのQRコード更新）
Parts:
- removed the G*** at (118.7, 79.3)
- added G***: LOGO, GPS_TFT:QRv7, B.Cu at (119.0, 78.9)
- SW1: moved to B.Cu
- moved SW1 4.48 mm to (74.7, 100.4), turned to -90 degrees
- moved R53 2.19 mm to (115.9, 89.2)
Routing:
- net Net-(U10-H_CSN): track 9.06 -> 11.3 mm
- net SPI1_CS: track 44.6 -> 42.3 mm
- net GND: track 294.6 -> 293.0 mm, vias 60 -> 61
- net SW_TOGGLE: track 42.1 -> 43.6 mm
