File: kicad/mainboard/DisplayModule_PONSv7.kicad_sch (KiCad schematic)
At the start: 55 parts, among them J1 Ext. Speaker, J10 Conn_01x05_MountingPin, J2 Conn_01x04_MountingPin, J4 Micro_SD_Card_Det2, J5 2005280040, J6 54132-4062, J9 Conn_01x04_MountingPin, SW1 PTS645Vx58-2, U1 MS5611-01BA, U4 PAM8302AAD

Commit message: 0.960 ソフトウェア＋ドキュメント KiCad v7 基板
普段編集しないモジュールを src/ へ移動し、README を v7 に更新

■ src/ への移動（Arduino IDE のタブ削減）
Arduino IDE はスケッチ直下のファイルを全部タブに出すため 28 個まで増え、
目的のファイルを探しづらくなっていた。仕様が固まっていて普段いじらない
4 モジュールを src/ へ移し、タブを 20 個に減らした。

  src/button.*     ボタン入力・メニュー
  src/sound.*      音声出力（WAV・トーン）
  src/vectormap.*  ベクタ地図の描画
  src/imulog.*     生 IMU ロガー

src/ 配下もコンパイルされるが IDE のタブには出ない。裏を返すと IDE からは
編集できなくなるので、これらは VSCode 等で編集すること。
またスケッチ直下は include パスに入っていないため、src/ の中からルート側の
ヘッダを参照するときは "../mysd.h" のように 1 段戻る必要がある。
この経緯と注意点は GPS_TFT_map.ino のヘッダに残した。

#include は 27 箇所を書き換え、全 104 件が実在するパスへ解決することを確認。

■ 併せて修正
button.cpp の #include "Button.h" が大文字始まりだった。macOS は
ファイルシステムが大文字小文字を区別しないため通っていたが、Linux では
壊れる。"button.h" に修正。

■ README を v7 に更新
 * タイトルとスペックを v7 へ。ソフトウェアバージョン 0.942 → 0.960
 * PONS Link（機体⇄ボート テレメトリ無線）の節を新設。3 台構成、下り一方向に
   した理由、無線パラメータ、実測 350m。設計の詳細は docs/pons_link.md へ
 * BNO085 を β 試験版から標準搭載へ。SPI 接続にした理由も記載
 * マイコンを RP2350B（外付け FLASH 16MB）と明記
 * PCBA とは別に発注する部品の一覧表（Digikey / マルツ / 秋月）を追加
 * 警告音・SD ログ・使用部品に無線関連を追記

重量とバッテリー持続時間は v7 実機での計測待ちのため、v6 β版の参考値と
PONS Link の消費電流だけを記載した。水面での到達距離も未確認と明記。

普段編集しないモジュールを src/ へ移動し、README を v7 に更新

■ src/ への移動（Arduino IDE のタブ削減）
Arduino IDE はスケッチ直下のファイルを全部タブに出すため 28 個まで増え、
目的のファイルを探しづらくなっていた。仕様が固まっていて普段いじらない
4 モジュールを src/ へ移し、タブを 20 個に減らした。

  src/button.*     ボタン入力・メニュー
  src/sound.*      音声出力（WAV・トーン）
  src/vectormap.*  ベクタ地図の描画
  src/imulog.*     生 IMU ロガー

src/ 配下もコンパイルされるが IDE のタブには出ない。裏を返すと IDE からは
編集できなくなるので、これらは VSCode 等で編集すること。
またスケッチ直下は include パスに入っていないため、src/ の中からルート側の
ヘッダを参照するときは "../mysd.h" のように 1 段戻る必要がある。
この経緯と注意点は GPS_TFT_map.ino のヘッダに残した。

#include は 27 箇所を書き換え、全 104 件が実在するパスへ解決することを確認。

■ 併せて修正
button.cpp の #include "Button.h" が大文字始まりだった。macOS は
ファイルシステムが大文字小文字を区別しないため通っていたが、Linux では
壊れる。"button.h" に修正。

■ README を v7 に更新
 * タイトルとスペックを v7 へ。ソフトウェアバージョン 0.942 → 0.960
 * PONS Link（機体⇄ボート テレメトリ無線）の節を新設。3 台構成、下り一方向に
   した理由、無線パラメータ、実測 350m。設計の詳細は docs/pons_link.md へ
 * BNO085 を β 試験版から標準搭載へ。SPI 接続にした理由も記載
 * マイコンを RP2350B（外付け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
Parts:
- removed C39: 100n, GPS_TFT:C_0402_1005Metric_small_pads, symbol Device:C
- removed J10: Conn_01x05_MountingPin, Connector_JST:JST_SHL_SM06B-SHLS-TF_1x06-1MP_P1.00mm_Horizontal, symbol Connector_Generic_MountingPin:Conn_01x06_MountingPin
- removed J2, J9: Conn_01x04_MountingPin, Connector_JST:JST_SH_SM04B-SRSS-TB_1x04-1MP_P1.00mm_Horizontal, symbol Connector_Generic_MountingPin:Conn_01x04_MountingPin
- removed JP1: TFT_JMP, Jumper:SolderJumper-2_P1.3mm_Open_RoundedPad1.0x1.5mm, symbol Jumper:SolderJumper_2_Open
- removed R2: 470, Resistor_SMD:R_0402_1005Metric, symbol Device:R
- removed R20: 4.7k, Resistor_SMD:R_0402_1005Metric, symbol Device:R
- removed SW1: PTS645Vx58-2, Button_Switch_THT:SW_Tactile_SPST_Angled_PTS645Vx58-2LFS, symbol Switch:SW_Push
- removed U1: MS5611-01BA, Package_LGA:LGA-8_3x5mm_P1.25mm, symbol Sensor_Pressure:MS5611-01BA
- added C11: 100n, GPS_TFT:C_0402_1005Metric_small_pads, symbol Device:C
- added R6: 100K, Resistor_SMD:R_0402_1005Metric, symbol Device:R
- added R7: 10k, Resistor_SMD:R_0603_1608Metric_Pad0.98x0.95mm_HandSolder, symbol Device:R
- added U2: W25Q128JVS, Package_SO:SOIC-8_5.3x5.3mm_P1.27mm, symbol Memory_Flash:W25Q128JVS
- FB1: renamed from FB2; now in the parts list
- FB2: renamed from FB1; now in the parts list
- J3: renamed from J5; now in the parts list
- R10: renamed from R3; footprint Resistor_SMD:R_0603_1608Metric -> Resistor_SMD:R_0402_1005Metric; LCSC C23179 -> C25117
- R11: renamed from R1; footprint Resistor_SMD:R_0603_1608Metric -> Resistor_SMD:R_0402_1005Metric; LCSC C23179 -> C25117
- R12: renamed from R11; value 47 -> 33; footprint Resistor_SMD:R_0603_1608Metric -> Resistor_SMD:R_0402_1005Metric; LCSC C23182 -> C25105
- R13: renamed from R12; value 47 -> 33; footprint Resistor_SMD:R_0603_1608Metric -> Resistor_SMD:R_0402_1005Metric; LCSC C23182 -> C25105
- R14: renamed from R13; value 47 -> 33; footprint Resistor_SMD:R_0603_1608Metric -> Resistor_SMD:R_0402_1005Metric; LCSC C23182 -> C25105
- R15: renamed from R14; value 47 -> 33; footprint Resistor_SMD:R_0603_1608Metric -> Resistor_SMD:R_0402_1005Metric; LCSC C23182 -> C25105
- R16: renamed from R15; value 47 -> 33; footprint Resistor_SMD:R_0603_1608Metric -> Resistor_SMD:R_0402_1005Metric; LCSC C23182 -> C25105
- R17: renamed from R16; value 47 -> 33; footprint Resistor_SMD:R_0603_1608Metric -> Resistor_SMD:R_0402_1005Metric; LCSC C23182 -> C25105
- U1: renamed from U4; value PAM8302AAD -> PAM8302AADCR
- renumbered C8 to C1, C12 to C10, C1 to C12, C3 to C13, C4 to C14, C6 to C2, C5 to C3, C13 to C4, C10 to C5, C7 to C6, C9 to C7, C11 to C8, C15 to C9, D5 to D1, J6 to J2, R38 to R1, R7 to R18, R17 to R19, R37 to R2, R18 to R20, R19 to R21, R21 to R22, R22 to R23, R10 to R3, R9 to R4, R8 to R5, R4 to R9
Connections:
- net +3V3: now also C11.1, R7.1, U2.8 (VCC)
- net AMP_SD: now also R6.1
- net GND: now also J4.SH (SHIELD), C11.2, R6.2, U2.4 (GND); no longer J4.11 (SHIELD)
- new net QSPI_SCLK: U2.6 (CLK)
- new net QSPI_SD0: U2.5 (DI/IO_{0})
- new net QSPI_SD1: U2.2 (DO/IO_{1})
- new net QSPI_SD2: U2.3 (~{WP}/IO_{2})
- new net QSPI_SD3: U2.7 (~{HOLD}/~{RESET}/IO_{3})
- new net QSPI_SS: R7.2, U2.1 (~{CS})
- no-connect marks 9 -> 8
Other:
- sheet RP2354B renamed RP2350B
- added sheet PERIPHERAL (MS5611BNO085.kicad_sch)
- note added: "(3.3V-2.0V)/200 Ohm=6.5mA"
- note added: "(5V-3.0V)/470 Ohm =4.2mA"
- note added: "BLM31PG391SN1L"
- note added: "FLASH"
- note added: "[Memo JLCPCB BOM Exemption] J1 Speaker socket (No parts required) J5 Debug SH 3p(No use. Debug purpose) U12 E220 LoRa (Due to 技適, 手実装) U6,U7 CUS-12TB Switch (JLCPCBにないパーツのため手実装） H1,H2,H3,H4 Hole TP3 LoRa JP"
- note removed: "(3.3V-2.0V)/200Ohm=6.5mA"
- note removed: "(5V-3.0V)/47Ohm=4.2mA"
- note removed: "BLM31PG121SN1L"
- note removed: "I2C address select"
- note removed: "Memo JLCPCB BOM Exemption molex 40p PWR1 JST PH 2P FB1,FB2 Ferrite beads J1 Speaker socket(No parts) J2 SH 4p UART2 J5 UART Molex J6 40p molex J7 Debug SH 3p J8 I2C SH 4p J9 SH 4p UART Backup SW1 Vertical Toggle SW Tactile SW 434133025816 MicroSD card slot micro USB-B MS5611 Airdata MCP73831 Charge PAM8302 Audio"
- title: PONS for HPA v6 -> PONS for HPA v7
- moved on the sheet: C1, C4, D1, D2, H1, H2, H3, H4, R11, R18
