File: kicad/mainboard/MS5611BNO085.kicad_sch (KiCad schematic)
At the start: 28 parts, among them U10 BNO085, U12 E220-900T22S(JP), U8 MS5611-01BA, Y2 32.768k

Commit message: kicadデータ更新
KiCad プロジェクトを自己完結化（ライブラリテーブルと独自シンボルの取り込み）

クローンしただけでは GPS_TFT: などのライブラリが解決できず、また一部の
シンボルが KiCad 標準ライブラリ本体を書き換えて作られていたため、他の環境
では正しく再現できない状態だった。プロジェクト内で完結するよう整理した。

■ ライブラリテーブルを追加
fp-lib-table / sym-lib-table がリポジトリに一度も入っていなかった。
3 プロジェクト分を ${KIPRJMOD} 相対で新規作成。絶対パスを使っていないので
どこへ置いても、どのマシンでも解決する。
回路図が別名で参照している nickname（2005280040 / 54132-4062 / CUS-12TB /
RP2350_80QFN_minimal）も同じフォルダを指すよう登録した。

■ 標準ライブラリへの依存を解消
6 つの標準ライブラリがローカルで書き換えられていた（codesign --verify で
確認）。使用中のシンボルを上流 kicad-symbols 10.0.6 と 1 つずつ比較し、
差があるものだけプロジェクト内へ移した。

  追加されていたもの
    RF_Module:E220-900T22S(JP)  → E220-900T22S:E220-900T22S(JP)
    Sensor_Motion:BNO085        → bno085:BNO085
    Switch:CUS-12TB             → CUS-12TB:CUS-12TB

  公式シンボルを改変していたもの（ピン番号が変わるため影響が大きい）
    Connector:USB_B_Micro       → USB_microB:USB_B_Micro
      上流は 1-5,SH。手元はシールドパッドのピン 6 を追加した版
    Connector_Generic_Shielded:Conn_01x03_Shielded
                                → Conn_01x03_Shielded:Conn_01x03_Shielded
      上流はシールドピンが SH。手元は MP に改名した版

  上流と一致していたもの（標準ライブラリのまま参照する）
    Conn_01x02_Pin / Conn_01x04_Pin / Micro_SD_Card_Det2 /
    TestPoint_2Pole / SW_Push

改変版と上流の差は sym-lib-table の descr に書いてある。

■ 整理
 * DMG3415U.kicad_sym は中身が DMP2045 だったので dmp2045.kicad_sym へ改名
   （回路図の参照 dmp2045:DMP2045 が切れていたのを修復）
 * 未使用のフットプリント 6 件とシンボル 5 件を削除
 * .gitignore のパターンがプロジェクト名を直書きしていて v7 のバックアップ
   フォルダに当たっていなかったため、*-backups/ 等の総称に変更

回路図の lib_id を貼り替えただけで、シンボル本体・ピン・フットプリント指定は
変えていない。ネットリストと部品構成に変更はなく、発注済みの基板データにも
影響しない。全 158 件の参照が解決することを確認済み。
Parts:
- U10: symbol Sensor_Motion:BNO085 -> bno085:BNO085
- U12: symbol RF_Module:E220-900T22S(JP) -> E220-900T22S:E220-900T22S(JP)
Changed lines of the file:
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@@
 	)
 	(symbol
-		(lib_id "Sensor_Motion:BNO085")
+		(lib_id "bno085:BNO085")
 		(at 135.89 46.99 0)
 		(unit 1)
@@
 	)
 	(symbol
-		(lib_id "RF_Module:E220-900T22S(JP)")
+		(lib_id "E220-900T22S:E220-900T22S(JP)")
 		(at 59.69 149.86 0)
 		(unit 1)
