File: kicad/mainboard/MS5611BNO085.kicad_sch (KiCad schematic)
At the start: 22 parts, among them J6 Conn_01x08_MountingPin, J7 2005280050, J8 2005280040, U8 MS5611-01BA, U9 E220-900T22S(JP)

Commit message: 0.994 GNSS の翌日起動を速くし、本番前チェック・高温充電の警告・電池低下の点滅を入れ、v7.1 基板の逆接保護と発注前の修正を仕上げた
- GNSS: AssistNow Autonomous を有効化（CFG-VALSET で RAM と BBR。settings.h の
  GNSS_USE_ANA。0 でも OFF を書き込む＝BBR に残った ON を消すため）。前日と同じ時間帯の
  起動が 23〜28 秒 → 3〜4 秒（BT1 が生きていること）。NAV-AOPSTATUS を 1Hz で受け、
  GNSS DETAIL 3 に ANA:ON data/use/calc、log.txt に「... after boot」（TTFF）・最初の
  測位の軌道の出どころ・10 分ごとの計算時間。ACK 待ちの間も imu_service_if_due() を
  呼ぶ（以前からの抜け）
- readiness.cpp（新規）: 本番前チェック。GNSS・IMU・ESKF・較正（マウント外れだけ。
  日付またぎは推測なので入れない＝台の上での APPLY を促さない）・地上の姿勢・設定画面の
  赤丸・USB・電池 50%・SD・無線（送信モード）がそろい、地上で止まっていたら 1 度だけ
  「準備完了」（ready.wav）。欠けていれば設定画面の右上に項目名。受信モード・リプレイ・
  デモは対象外。既存の判定を読むだけで、条件は書き写さない
- 高温での充電の警告（v7・v7.1）: USB 接続中に MS5611 が 45°C を 30 秒超え続けたら
  地図に TOO HOT TO CHARGE と charge_hot.wav（60 秒ごと・最低音量 60）。電池の仕様は
  充電 0〜45°C。地図の段は電源異常と共用（異常 ＞ 高温 ＞ SW OFF）
- 電池低下のときの点滅（v7.1）: 電池低下の警告と同じ 3.5V でバックライトを 2 秒点灯・
  4 秒消灯。3.65V か USB で戻る（3.5V で戻すと入り切りをくり返す）。消灯中も本来の
  明るさは追い続ける（照度追従の立ち上がりで 2 秒の点灯が暗くならないように）
- 本体の回路図・PCB: 電池の逆接保護 Q4（AO3401A、D が電池側）＋ R52、PWR1 の
  ネットを VBAT_RAW に。C32 を 10µF 0805 に（10/20 に直したのが 0402 に戻っていた）。
  D5 を RB751S40（逆流が少ない。PCBA で実装）に。古いメモを整理
- IMU 基板の GND が IC1.16・C3 だけ分かれていたのをつないだ。J3 の値を 01x08 に。
  case_cover の部品番号を回路図と一致。GNSS 基板の裏面を GND ベタに（浮いていた
  19 個のビアがつながった）
- 音声 2 本（ready / charge_hot）は macOS の音声合成の仮音声
- docs: pons_power.md に Q4・P-ch FET 3 段の役割・電池の保護回路（DTP603048(PHR) の
  仕様書）・R39 を 2.2kΩ に戻さない理由（電池の最大充電 430mA も超える）・高温の警告・
  電池低下の点滅。README に GNSS の起動・本番前チェック・新しい警報・v7.1 の USB-C と
  充電時間、古い記述（v7 の実結線試験・無線の立ち上げ手順書の冒頭）を今の状態に。
  CLAUDE.md に BBR に書いた GNSS 設定が残る件と readiness.cpp
- kicad/.gitignore に *.pos

PONS_BOARD は V7 と V71 の両方でビルド OK（4,052,376 / 4,046,728 B）/
gen_wav_flash.py --check は 37 ファイル一致 / 本体 PCB の DRC は未配線 0・回路図と一致
（シルクの 6 件は意図どおり）/ IMU・カバー・GNSS 基板も未配線 0・回路図と一致 /
BOM の LCSC 番号は全 48 種類を JLC/LCSC の部品情報と照合 / 実機は未確認

Co-Authored-By: Claude Opus 5.5 <noreply@anthropic.com>
Parts:
- D5: value RB520S-30 -> RB751S40; LCSC (none) -> C232576; now in the parts list
- U8: FT Rotation Offset (none) -> 90
Other:
- note added: "BT1が放電しきっていても、即座にGNSSが起動できる電圧をV_BCKUPに提供する V_BCKP Minimum operating voltage = 1.65V 抵抗によって、BT1バッテリーが空っぽでも、V_BCKUPに電圧が生じる((3.3-0.6)*470/690)=1.8Vぐらい 放電時の電圧降下はV=IR=10*10^-6*470 で、電圧降下はほとんどない P=IV=V^2/R=(0.5*10^-3)^2/500=0.5*10^-9=0.5nW"
- note removed: "BT1が放電しきっていると、モジュールが起動しないバグがあった。 V_BCKP Minimum operating voltage = 1.65V R2抵抗によって、BT1バッテリーが空っぽでも、V_BCKUPに電圧が生じる((3.3-0.6)*470/690)=1.8Vぐらい 放電時は、R2の電圧降下はV=IR=10*10^-6*470 で、電圧降下はほとんどない P=IV=V^2/R=(0.5*10^-3)^2/500=0.5*10^-9=0.5nW"
- note removed: "M0,M1 ピン変更あり"
- moved on the sheet: R41, R42
Changed lines of the file:
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@@
 	(title_block
 		(title "PONS for HPA v7")
-		(date "2026-09-06")
-		(rev "7.0")
+		(date "2026-10-22")
+		(rev "7.1")
 		(comment 1 "GNSS, SD, Speaker, Lipo Charger")
 		(comment 2 "Good for outdoor use with high brightness")
@@
 	(rectangle
 		(start 15.24 107.95)
-		(end 128.016 186.055)
+		(end 115.316 186.055)
 		(stroke
 			(width 0)
@@
 		)
 	)
-	(text "BT1が放電しきっていると、モジュールが起動しないバグがあった。\nV_BCKP Minimum operating voltage = 1.65V\nR2抵抗によって、BT1バッテリーが空っぽでも、V_BCKUPに電圧が生じる((3.3-0.6)*470/690)=1.8Vぐらい\n放電時は、R2の電圧降下はV=IR=10*10^-6*470 で、電圧降下はほとんどない\nP=IV=V^2/R=(0.5*10^-3)^2/500=0.5*10^-9=0.5nW"
+	(text "BT1が放電しきっていても、即座にGNSSが起動できる電圧をV_BCKUPに提供する\nV_BCKP Minimum operating voltage = 1.65V\n抵抗によって、BT1バッテリーが空っぽでも、V_BCKUPに電圧が生じる((3.3-0.6)*470/690)=1.8Vぐらい\n放電時の電圧降下はV=IR=10*10^-6*470 で、電圧降下はほとんどない\nP=IV=V^2/R=(0.5*10^-3)^2/500=0.5*10^-9=0.5nW"
 		(exclude_from_sim no)
-		(at 190.5 157.734 0)
+		(at 184.912 158.242 0)
 		(effects
 			(font
@@
 		(effects
 			(font
-				(size 1.27 1.27)
+				(size 2.54 2.54)
+				(thickness 0.508)
+				(bold yes)
 			)
 		)
@@
 		)
 	)
-	(text "M0,M1 ピン変更あり"
-		(exclude_from_sim no)
-		(at 99.06 183.896 0)
-		(effects
-			(font
-				(size 10 10)
-			)
-		)
-	)
 	(text "EXTERNAL CONNECTORS"
 		(exclude_from_sim no)
@@
 		(effects
 			(font
-				(size 1.27 1.27)
+				(size 2.54 2.54)
+				(thickness 0.508)
+				(bold yes)
 			)
+			(justify left)
 		)
 	)
 	(text "MS5611"
 		(exclude_from_sim no)
-		(at 22.86 18.034 0)
+		(at 17.526 18.796 0)
 		(effects
 			(font
-				(size 1.27 1.27)
+				(size 2.54 2.54)
+				(thickness 0.508)
+				(bold yes)
 			)
+			(justify left)
 		)
 	)
@@
 	(wire
 		(pts
-			(xy 67.31 93.98) (xy 67.31 87.63)
+			(xy 152.4 179.07) (xy 152.4 172.72)
 		)
 		(stroke
@@
 	(wire
 		(pts
-			(xy 67.31 77.47) (xy 67.31 80.01)
+			(xy 152.4 162.56) (xy 152.4 165.1)
 		)
 		(stroke
@@
 	(wire
 		(pts
-			(xy 72.39 77.47) (xy 72.39 80.01)
+			(xy 157.48 162.56) (xy 157.48 165.1)
 		)
 		(stroke
@@
 	(wire
 		(pts
-			(xy 54.61 96.52) (xy 72.39 96.52)
+			(xy 139.7 181.61) (xy 157.48 181.61)
 		)
 		(stroke
@@
 	(wire
 		(pts
-			(xy 54.61 93.98) (xy 67.31 93.98)
+			(xy 139.7 179.07) (xy 152.4 179.07)
 		)
 		(stroke
@@
 	(wire
 		(pts
-			(xy 72.39 96.52) (xy 72.39 87.63)
+			(xy 157.48 181.61) (xy 157.48 172.72)
 		)
 		(stroke
@@
 	(global_label "I2C0_SDA"
 		(shape input)
-		(at 54.61 96.52 180)
+		(at 139.7 181.61 180)
 		(fields_autoplaced yes)
 		(effects
@@
 		)
 		(property "Intersheetrefs" "${INTERSHEET_REFS}"
-			(at 42.7953 96.52 0)
+			(at 127.8853 181.61 0)
 			(hide yes)
 			(show_name no)
@@
 	(global_label "I2C0_SCL"
 		(shape input)
-		(at 54.61 93.98 180)
+		(at 139.7 179.07 180)
 		(fields_autoplaced yes)
 		(effects
@@
 		)
 		(property "Intersheetrefs" "${INTERSHEET_REFS}"
-			(at 42.8558 93.98 0)
+			(at 127.9458 179.07 0)
 			(hide yes)
 			(show_name no)
@@
 		(lib_name "+3V3_2")
 		(lib_id "power:+3V3")
-		(at 67.31 77.47 0)
+		(at 152.4 162.56 0)
 		(unit 1)
 		(body_style 1)
@@
 		(dnp no)
 		(property "Reference" "#PWR088"
-			(at 67.31 81.28 0)
+			(at 152.4 166.37 0)
 			(hide yes)
 			(show_name no)
@@
 		)
 		(property "Value" "+3V3"
-			(at 66.802 73.66 0)
+			(at 151.892 158.75 0)
 			(show_name no)
 			(do_not_autoplace no)
@@
 		)
 		(property "Footprint" ""
-			(at 67.31 77.47 0)
+			(at 152.4 162.56 0)
 			(hide yes)
 			(show_name no)
@@
 		)
 		(property "Datasheet" ""
-			(at 67.31 77.47 0)
+			(at 152.4 162.56 0)
 			(hide yes)
 			(show_name no)
@@
 		)
 		(property "Description" "Power symbol creates a global label with name \"+3V3\""
-			(at 67.31 77.47 0)
+			(at 152.4 162.56 0)
 			(hide yes)
 			(show_name no)
@@
 			)
 		)
+		(property "FT Rotation Offset" "90"
+			(at 52.07 44.45 0)
+			(hide yes)
+			(show_name no)
+			(do_not_autoplace no)
+			(effects
+				(font
+					(size 1.27 1.27)
+				)
+			)
+		)
 		(pin "2"
 		)
@@
 	(symbol
 		(lib_id "Device:R")
-		(at 72.39 83.82 0)
+		(at 157.48 168.91 0)
 		(unit 1)
 		(body_style 1)
@@
 		(dnp no)
 		(property "Reference" "R42"
-			(at 70.358 83.82 90)
+			(at 155.448 168.91 90)
 			(show_name no)
 			(do_not_autoplace no)
@@
 		)
 		(property "Value" "4.7k"
-			(at 72.39 83.82 90)
+			(at 157.48 168.91 90)
 			(show_name no)
 			(do_not_autoplace no)
@@
 		)
 		(property "Footprint" "Resistor_SMD:R_0402_1005Metric"
-			(at 70.612 83.82 90)
+			(at 155.702 168.91 90)
 			(hide yes)
 			(show_name no)
@@
 		)
 		(property "Datasheet" ""
-			(at 72.39 83.82 0)
+			(at 157.48 168.91 0)
 			(hide yes)
 			(show_name no)
@@
 		)
 		(property "Description" ""
-			(at 72.39 83.82 0)
+			(at 157.48 168.91 0)
 			(hide yes)
 			(show_name no)
@@
 		)
 		(property "Sim.Device" ""
-			(at 72.39 83.82 90)
+			(at 157.48 168.91 90)
 			(hide yes)
 			(show_name no)
@@
 		)
 		(property "Sim.Type" ""
-			(at 72.39 83.82 90)
+			(at 157.48 168.91 90)
 			(hide yes)
 			(show_name no)
@@
 		)
 		(property "LCSC" "C25900"
-			(at 72.39 83.82 90)
+			(at 157.48 168.91 90)
 			(hide yes)
 			(show_name no)
@@
 	(symbol
 		(lib_id "Device:R")
-		(at 67.31 83.82 0)
+		(at 152.4 168.91 0)
 		(unit 1)
 		(body_style 1)
@@
 		(dnp no)
 		(property "Reference" "R41"
-			(at 65.278 83.82 90)
+			(at 150.368 168.91 90)
 			(show_name no)
 			(do_not_autoplace no)
@@
 		)
 		(property "Value" "4.7k"
-			(at 67.31 83.82 90)
+			(at 152.4 168.91 90)
 			(show_name no)
 			(do_not_autoplace no)
@@
 		)
 		(property "Footprint" "Resistor_SMD:R_0402_1005Metric"
-			(at 65.532 83.82 90)
+			(at 150.622 168.91 90)
 			(hide yes)
 			(show_name no)
@@
 		)
 		(property "Datasheet" ""
-			(at 67.31 83.82 0)
+			(at 152.4 168.91 0)
 			(hide yes)
 			(show_name no)
@@
 		)
 		(property "Description" ""
-			(at 67.31 83.82 0)
+			(at 152.4 168.91 0)
 			(hide yes)
 			(show_name no)
@@
 		)
 		(property "Sim.Device" ""
-			(at 67.31 83.82 90)
+			(at 152.4 168.91 90)
 			(hide yes)
 			(show_name no)
@@
 		)
 		(property "Sim.Type" ""
-			(at 67.31 83.82 90)
+			(at 152.4 168.91 90)
 			(hide yes)
 			(show_name no)
@@
 		)
 		(property "LCSC" "C25900"
-			(at 67.31 83.82 90)
+			(at 152.4 168.91 90)
 			(hide yes)
 			(show_name no)
@@
 		(body_style 1)
 		(exclude_from_sim no)
-		(in_bom no)
+		(in_bom yes)
 		(on_board yes)
 		(in_pos_files yes)
@@
 			)
 		)
-		(property "Value" "RB520S-30"
+		(property "Value" "RB751S40"
 			(at 247.65 126.9999 90)
 			(show_name no)
@@
 			)
 		)
-		(property "Datasheet" "http://www.vishay.com/docs/88503/1n4001.pdf"
+		(property "Datasheet" "https://www.onsemi.com/download/data-sheet/pdf/rb751s40t1-d.pdf"
 			(at 245.11 125.73 0)
 			(hide yes)
@@
 			)
 		)
-		(property "Description" "50V 1A General Purpose Rectifier Diode, DO-41"
+		(property "Description" "40 V SCHOTTKY BARRIER DIODE"
 			(at 245.11 125.73 0)
 			(hide yes)
@@
 			)
 		)
+		(property "LCSC" "C232576"
+			(at 245.11 125.73 90)
+			(hide yes)
+			(show_name no)
+			(do_not_autoplace no)
+			(effects
+				(font
+					(size 1.27 1.27)
+				)
+			)
+		)
 		(pin "1"
 		)
@@
 		(lib_name "+3V3_2")
 		(lib_id "power:+3V3")
-		(at 72.39 77.47 0)
+		(at 157.48 162.56 0)
 		(unit 1)
 		(body_style 1)
@@
 		(dnp no)
 		(property "Reference" "#PWR089"
-			(at 72.39 81.28 0)
+			(at 157.48 166.37 0)
 			(hide yes)
 			(show_name no)
@@
 		)
 		(property "Value" "+3V3"
-			(at 71.882 73.66 0)
+			(at 156.972 158.75 0)
 			(show_name no)
 			(do_not_autoplace no)
@@
 		)
 		(property "Footprint" ""
-			(at 72.39 77.47 0)
+			(at 157.48 162.56 0)
 			(hide yes)
 			(show_name no)
@@
 		)
 		(property "Datasheet" ""
-			(at 72.39 77.47 0)
+			(at 157.48 162.56 0)
 			(hide yes)
 			(show_name no)
@@
 		)
 		(property "Description" "Power symbol creates a global label with name \"+3V3\""
-			(at 72.39 77.47 0)
+			(at 157.48 162.56 0)
 			(hide yes)
 			(show_name no)
