File: kicad/mainboard/SHT_RP2354B.kicad_sch (KiCad schematic)
At the start: 56 parts, among them J5 Conn_01x03_Shielded, J6 USB_B_Micro, Q1 AO3401A, SW1 PTS645VK392LFS, SW2 SW_TS-1088, SW3 SW_TS-1088, U3 RP2350_80QFN, U4 MCP73831-2-OT, U5 TPS63031DSK, U6 MAINSW_CUS-12TB, U7 TFTSW_CUS-12TB, Y1 X322512MSB4SI

Commit message: 0.962 KiCad 更新、production を git 管理から外す
fabrication-toolkit が生成する production/ は発注のたびに作り直せるうえ、
基板を直すたびに巨大な差分になるので .gitignore に追加した。

Co-Authored-By: Claude Opus 5 <noreply@anthropic.com>
Parts:
- SW1: now left out of the parts list
Changed lines of the file:
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@@
 		(body_style 1)
 		(exclude_from_sim no)
-		(in_bom yes)
+		(in_bom no)
 		(on_board yes)
 		(in_pos_files yes)

Commit message: 0.986 新基板（SCH16T 外付け）の kicad を追加し、ガーバー出力を git から外した
kicad/IMU_murata/ — SCH16T-K01-10 のブレイクアウト（新規）
本体の J7（Molex 200528-0080・8pin FPC）へ 1:1 ケーブルで繋ぐ外付け基板。
J1 のピン順を本体 J7 と一致させてある（1=+3V3 2=RESET 3=MOSI 4=CS 5=SCK
6=SYNC 7=MISO 8=GND）。シンボルとフットプリントも同梱。
- ★ R2（CS-GND の 4.7k）は実装しない。CS は負論理なので、プルダウンすると
  MCU が駆動していない間セレクト状態になる。R1（EXTRESN プルアップ）は実装する
- 本体側の GPIO 割り当ては settings.h の SCH16T_PIN_* が正本
  （一覧は docs/imu_sch16t_plan.md §3）

mainboard / GNSS モジュールの更新
- mainboard: DisplayModule_PONSv7 の pcb / pro / sch、MS5611BNO085.kicad_sch、
  SHT_RP2354B.kicad_sch
- GNSS モジュール: pcb / pro / sch、および QRv7 と FPC 4p のフットプリントを
  同プロジェクトの Footprints/ へ取り込み

kicad/FPC/ を畳んだ
FPC コネクタ 1 個のためのプロジェクトだったので、フットプリントを
kicad/GNSSboard_SAM-M10Q/Footprints/ へ移して削除した。
中身は同じで、差分は KiCad が再生成する uuid だけ。

ガーバー・ドリルのプロット出力を git から外した
kicad/.gitignore に追加（*.gbr *.gbl *.gbs *.gbp *.gbo *.gm1 *.gtl *.gts
*.gtp *.gto *.drl と、保険の *plot/ *plot.zip）。発注のたびに作り直せるうえ、
基板を直すたびに巨大な差分になる（ルート .gitignore の production/ と同じ理由）。
★ 入れ物のフォルダ名で書かないこと。v5_1plot/ のような名前は付け方が毎回違うので
  次の基板で外れる。既存の *-backups/ / *.kicad_prl と同じ方針。

Co-Authored-By: Claude Opus 5 <noreply@anthropic.com>
Connections:
- net PWR_TFT is gone; now on net TFT_SW: U7.P$2 (2)
- net BNO_INT renamed SCH16T_RESET
- net BNO_NRST renamed SCH16T_SYNC
- net BNO_WAKE renamed LORA_M01
- net I2C1_SCL renamed TFT_SW
- net I2C1_SDA renamed TFT_MOSFET_G
Other:
- note added: "E220 M01 移動"
- note removed: "移動 10->34"
- note removed: "移動 11->35"
Changed lines of the file:
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@@
 		)
 	)
-	(text "移動 10->34"
-		(exclude_from_sim no)
-		(at 160.782 155.702 0)
-		(effects
-			(font
-				(size 1.27 1.27)
-			)
-		)
-	)
 	(text "Modyfied"
 		(exclude_from_sim no)
@@
 		)
 	)
-	(text "移動 11->35"
+	(text "BAT IN"
 		(exclude_from_sim no)
-		(at 160.528 157.734 0)
+		(at 187.706 37.846 0)
 		(effects
 			(font
@@
 		)
 	)
-	(text "BAT IN"
+	(text "Grounding P-Ch FET Gate float\nat the same time"
 		(exclude_from_sim no)
-		(at 187.706 37.846 0)
+		(at 192.278 161.036 0)
 		(effects
 			(font
@@
 		)
 	)
-	(text "Grounding P-Ch FET Gate float\nat the same time"
+	(text "E220 M01 移動"
 		(exclude_from_sim no)
-		(at 192.278 161.036 0)
+		(at 151.13 193.04 0)
 		(effects
 			(font
@@
 		)
 	)
-	(global_label "PWR_TFT"
+	(global_label "TFT_SW"
 		(shape input)
 		(at 262.89 57.15 180)
@@
 		)
 		(property "Intersheetrefs" "${INTERSHEET_REFS}"
-			(at 251.922 57.15 0)
+			(at 253.2525 57.15 0)
 			(hide yes)
 			(show_name no)
@@
 		)
 	)
+	(global_label "TFT_MOSFET_G"
+		(shape input)
+		(at 143.51 154.94 0)
+		(fields_autoplaced yes)
+		(effects
+			(font
+				(size 1.27 1.27)
+			)
+			(justify left)
+		)
+		(property "Intersheetrefs" "${INTERSHEET_REFS}"
+			(at 159.9208 154.94 0)
+			(hide yes)
+			(show_name no)
+			(do_not_autoplace no)
+			(effects
+				(font
+					(size 1.27 1.27)
+				)
+				(justify left)
+			)
+		)
+	)
 	(global_label "USR_LED"
 		(shape input)
@@
 		)
 	)
-	(global_label "BNO_INT"
+	(global_label "TFT_SW"
 		(shape input)
-		(at 143.51 185.42 0)
+		(at 143.51 157.48 0)
 		(fields_autoplaced yes)
 		(effects
@@
 		)
 		(property "Intersheetrefs" "${INTERSHEET_REFS}"
-			(at 154.2967 185.42 0)
+			(at 153.1475 157.48 0)
 			(hide yes)
 			(show_name no)
@@
 		)
 	)
+	(global_label "SCH16T_SYNC"
+		(shape input)
+		(at 143.51 187.96 0)
+		(fields_autoplaced yes)
+		(effects
+			(font
+				(size 1.27 1.27)
+			)
+			(justify left)
+		)
+		(property "Intersheetrefs" "${INTERSHEET_REFS}"
+			(at 159.558 187.96 0)
+			(hide yes)
+			(show_name no)
+			(do_not_autoplace no)
+			(effects
+				(font
+					(size 1.27 1.27)
+				)
+				(justify left)
+			)
+		)
+	)
 	(global_label "QSPI_SS"
 		(shape input)
@@
 		)
 	)
+	(global_label "SCH16T_RESET"
+		(shape input)
+		(at 143.51 185.42 0)
+		(fields_autoplaced yes)
+		(effects
+			(font
+				(size 1.27 1.27)
+			)
+			(justify left)
+		)
+		(property "Intersheetrefs" "${INTERSHEET_REFS}"
+			(at 160.4045 185.42 0)
+			(hide yes)
+			(show_name no)
+			(do_not_autoplace no)
+			(effects
+				(font
+					(size 1.27 1.27)
+				)
+				(justify left)
+			)
+		)
+	)
 	(global_label "QSPI_SD3"
 		(shape input)
@@
 		)
 	)
-	(global_label "BNO_NRST"
-		(shape input)
-		(at 143.51 187.96 0)
-		(fields_autoplaced yes)
-		(effects
-			(font
-				(size 1.27 1.27)
-			)
-			(justify left)
-		)
-		(property "Intersheetrefs" "${INTERSHEET_REFS}"
-			(at 156.1714 187.96 0)
-			(hide yes)
-			(show_name no)
-			(do_not_autoplace no)
-			(effects
-				(font
-					(size 1.27 1.27)
-				)
-				(justify left)
-			)
-		)
-	)
 	(global_label "SW_TOGGLE"
 		(shape input)
@@
 		)
 	)
-	(global_label "I2C1_SCL"
-		(shape input)
-		(at 143.51 157.48 0)
-		(fields_autoplaced yes)
-		(effects
-			(font
-				(size 1.27 1.27)
-			)
-			(justify left)
-		)
-		(property "Intersheetrefs" "${INTERSHEET_REFS}"
-			(at 155.2642 157.48 0)
-			(hide yes)
-			(show_name no)
-			(do_not_autoplace no)
-			(effects
-				(font
-					(size 1.27 1.27)
-				)
-				(justify left)
-			)
-		)
-	)
-	(global_label "BNO_WAKE"
-		(shape input)
-		(at 143.51 190.5 0)
-		(fields_autoplaced yes)
-		(effects
-			(font
-				(size 1.27 1.27)
-			)
-			(justify left)
-		)
-		(property "Intersheetrefs" "${INTERSHEET_REFS}"
-			(at 156.3528 190.5 0)
-			(hide yes)
-			(show_name no)
-			(do_not_autoplace no)
-			(effects
-				(font
-					(size 1.27 1.27)
-				)
-				(justify left)
-			)
-		)
-	)
 	(global_label "DB7"
 		(shape input)
@@
 		)
 	)
-	(global_label "I2C1_SDA"
-		(shape input)
-		(at 143.51 154.94 0)
-		(fields_autoplaced yes)
-		(effects
-			(font
-				(size 1.27 1.27)
-			)
-			(justify left)
-		)
-		(property "Intersheetrefs" "${INTERSHEET_REFS}"
-			(at 155.3247 154.94 0)
-			(hide yes)
-			(show_name no)
-			(do_not_autoplace no)
-			(effects
-				(font
-					(size 1.27 1.27)
-				)
-				(justify left)
-			)
-		)
-	)
 	(global_label "DB2"
 		(shape input)
@@
 			(hide yes)
 			(show_name no)
+			(do_not_autoplace no)
+			(effects
+				(font
+					(size 1.27 1.27)
+				)
+				(justify left)
+			)
+		)
+	)
+	(global_label "LORA_M01"
+		(shape input)
+		(at 143.51 190.5 0)
+		(fields_autoplaced yes)
+		(effects
+			(font
+				(size 1.27 1.27)
+			)
+			(justify left)
+		)
+		(property "Intersheetrefs" "${INTERSHEET_REFS}"
+			(at 156.0504 190.5 0)
+			(hide yes)
+			(show_name no)

Commit message: 0.993 v7.1 基板の回路図と PCB を仕上げ、SW OFF のままの充電と電源異常を画面と音声で知らせるようにした
- power.cpp（新規）: USB の判定を usb_power_present() に一本化（v7.1 は VBUS を
  GPIO47 の ADC で測る）。電源経路の異常（2026-10-15 の充電 IC 焼損）を検出し、
  地図の POWER FAULT!! と power_fault.wav（30 秒ごと・最低音量 60）で知らせる。
  受信機は LINK_ST_PWR_FAULT を受けてトーン（同じ音声だとボートへの指示に聞こえる）
- v7.1: SW を OFF にしたまま USB で充電していると満充電にならない（Q3 のボディ
  ダイオード経由）。SW4 の OFF 側が GPIO40 を GND に落とすのを読み、地図に注意を出し
  1 度だけ読み上げる（charge_sw_off / charge_sw_on。排他グループ WAV_EXCL_CHARGE_SW）。
  移動中・ミラー中・リプレイ中・デモ中は出さない。判定に USB を入れない
  （VBUS が一瞬 4.3V を割ると 0V が本物の電池電圧として流れるため）。このあいだは
  電池低下の警告を止め、無線は RHAVE_VOLT を立てず LINK_ST_USB_SW_OFF、CSV は空欄
- 受信モードの電池表示を s55r42 の形に。SW OFF のまま USB の側は s5V / r5V
- backlight.cpp（新規）: v7.1 のバックライト PWM と VEML7700 の自動調光。
  飛行 CSV に lux / backlight 列
- E220 の M0/M1 は v7.1 で GPIO31 へ（GPIO47 は USB_SENS）
- 本体の回路図・PCB: SCH16T の J6 を逆順に（完成済みの FPC で J6-n ↔ J3-(9-n)）、
  F1 0805L035 → 0805L050（夏の充電で切れない）、R34/R35 を 10k/5.1k、C32 を 10µF 0805、
  SPI1 の SCK/MOSI/CS に 33Ω（R49〜R51）、スライドスイッチを MST-12D18G2 に、
  回路図とつながらない旧フットプリント（C33/R37/R38/R11 470Ω）を削除、DNP の BOM 除外、
  CUS-12TB の残骸とライブラリ登録を削除、メモの部品番号を v7.1 に
- GNSS 基板を 5 ピン（V_BCKUP）に。バックアップ電池は本体へ移した
- case_cover（照度センサー VEML7700）の kicad を追加。IMU ブレイクアウトの R2 を DNP
- 音声 3 本（power_fault / charge_sw_off / charge_sw_on）は macOS の音声合成の仮音声
- docs/pons_power.md（新規）。README の「自作の手順」を v7.1 に書き直し、
  SCH16T の配線の記述（J7・1:1 ケーブル）を J6・逆順に直した
- gen_wav_flash.py はコメント中の引用符付きの音声名も拾うので、録音前の名前を書かない

PONS_BOARD は V7 と V71 の両方でビルド OK（3,929,776 / 3,923,504 B）/
gen_wav_flash.py --check は 35 ファイル一致 / 本体 PCB の DRC は未配線 0・回路図と一致
（シルクの 6 件はボタンと USB の突起で意図どおり）/ GNSS 基板も未配線 0 / 実機は未確認

Co-Authored-By: Claude Opus 5.5 <noreply@anthropic.com>
Parts:
- removed C31: 4.7u, GPS_TFT:C_0402_1005Metric_small_pads, symbol Device:C
- removed C33: 100n, GPS_TFT:C_0402_1005Metric_small_pads, symbol Device:C
- removed C36, C37: 10u, GPS_TFT:C_0402_1005Metric_small_pads, symbol Device:C
- removed D3: 1N5819WS, Diode_SMD:D_SOD-323, symbol Diode:SS16
- removed D4: LED_R, LED_SMD:LED_0603_1608Metric_Pad1.05x0.95mm_HandSolder, symbol Device:LED
- removed J6: USB_B_Micro, Connector_USB:USB_Micro-B_Amphenol_10103594-0001LF_Horizontal, symbol USB_microB:USB_B_Micro
- removed L2: 1.5u, Inductor_SMD:L_APV_ANR3015, symbol Device:L
- removed Q1: AO3401A, Package_TO_SOT_SMD:SOT-23, symbol dmp2045:DMP2045
- removed R35: 5K1, Resistor_SMD:R_0402_1005Metric, symbol Device:R
- removed R36: 10K, Resistor_SMD:R_0402_1005Metric, symbol Device:R
- removed R39: 2.2k, Resistor_SMD:R_0402_1005Metric, symbol Device:R
- removed R42: 200, Resistor_SMD:R_0402_1005Metric, symbol Device:R
- removed U4: MCP73831-2-OT, Package_TO_SOT_SMD:SOT-23-5, symbol Battery_Management:MCP73831-2-OT
- removed U5: TPS63031DSK, Package_SON:WSON-10-1EP_2.5x2.5mm_P0.5mm_EP1.2x2mm, symbol Regulator_Switching:TPS63031DSK
- removed U6: MAINSW_CUS-12TB, GPS_TFT:CUS-12TB, symbol CUS-12TB:CUS-12TB
- removed U7: TFTSW_CUS-12TB, GPS_TFT:CUS-12TB, symbol CUS-12TB:CUS-12TB
- added C12: 100n, GPS_TFT:C_0402_1005Metric_small_pads, symbol Device:C
- added R48: 4.7k, Resistor_SMD:R_0402_1005Metric, symbol Device:R
- added R9: 10k, Resistor_SMD:R_0603_1608Metric_Pad0.98x0.95mm_HandSolder, symbol Device:R
- added SW5: MST-12D18G2 SMD SLIDE SWITCH, GPS_TFT:SW-SMD_3P-L9.1-W3.5-P2.50_MST-12D18G2, symbol Murata:MST-12D18G2SMDSLIDESWITCH
- added U2: W25Q128JVS, Package_SO:SOIC-8_5.3x5.3mm_P1.27mm, symbol Memory_Flash:W25Q128JVS
- L1: footprint GPS_TFT:L_pol_2016 -> Inductor_SMD:L_1008_2520Metric; LCSC C42411119 -> C22416628
- R32: renamed from R33; value 100K -> 100k
- SW3: renamed from SW1; now in the parts list
- renumbered C15 to C16, C16 to C17, C17 to C18, C18 to C19, C19 to C20, C20 to C21, C21 to C22, C22 to C23, C23 to C24, C24 to C25, C25 to C26, C26 to C27, C27 to C28, C28 to C29, C29 to C30, C30 to C31, C32 to C34, C34 to C36, C35 to C38, J5 to J4, R24 to R23, R25 to R24, R26 to R25, R27 to R26, R28 to R27, R29 to R28, R30 to R29, R31 to R30, R32 to R31, R34 to R33, R8 to R36, SW2 to SW1, SW3 to SW2
Connections:
- net +3V3: now also C12.1, R9.1, SW5.2, U2.8 (VCC)
- net GND: now also C12.2, R48.2, U2.4 (GND)
- net LORA_M01: now also U3.39 (GPIO31); no longer U3.58 (GPIO47_ADC7)
- net QSPI_SCLK: now also U2.6 (CLK)
- net QSPI_SD0: now also U2.5 (DI/IO_{0})
- net QSPI_SD1: now also U2.2 (DO/IO_{1})
- net QSPI_SD2: now also U2.3 (~{WP}/IO_{2})
- net QSPI_SD3: now also U2.7 (~{HOLD}/~{RESET}/IO_{3})
- net QSPI_SS: now also R9.2, U2.1 (~{CS})
- net TFT_SW: now also R48.1, SW5.1
- net USB_SENS: now also U3.58 (GPIO47_ADC7); no longer U3.39 (GPIO31)
- net ADC0: now reaches C28.1, R32.2, R33.1, U3.49 (GPIO40_ADC0)
- net VSYS renamed BATPWR
- no-connect marks 3 -> 1
Other:
- note added: "FLASH"
- note added: "移動 31->47"
- note added: "移動 47->31"
- note removed: "(5V-2.0V)/200Ohm=15mA"
- note removed: "2.2k to limit current"
- note removed: "Bat Discharger For Battery Safety"
- note removed: "GPIO pin changed"
- note removed: "Grounding P-Ch FET Gate float at the same time"
- note removed: "Power"
- note removed: "Power SW"
- note removed: "USB to Lipo Charger"
- moved on the sheet: C16, C17, C18, C19, C20, C21, C22, C23, C24, C25, C26, C27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

Commit message: 0.994 GNSS の翌日起動を速くし、本番前チェック・高温充電の警告・電池低下の点滅を入れ、v7.1 基板の逆接保護と発注前の修正を仕上げた
- GNSS: AssistNow Autonomous を有効化（CFG-VALSET で RAM と BBR。settings.h の
  GNSS_USE_ANA。0 でも OFF を書き込む＝BBR に残った ON を消すため）。前日と同じ時間帯の
  起動が 23〜28 秒 → 3〜4 秒（BT1 が生きていること）。NAV-AOPSTATUS を 1Hz で受け、
  GNSS DETAIL 3 に ANA:ON data/use/calc、log.txt に「... after boot」（TTFF）・最初の
  測位の軌道の出どころ・10 分ごとの計算時間。ACK 待ちの間も imu_service_if_due() を
  呼ぶ（以前からの抜け）
- readiness.cpp（新規）: 本番前チェック。GNSS・IMU・ESKF・較正（マウント外れだけ。
  日付またぎは推測なので入れない＝台の上での APPLY を促さない）・地上の姿勢・設定画面の
  赤丸・USB・電池 50%・SD・無線（送信モード）がそろい、地上で止まっていたら 1 度だけ
  「準備完了」（ready.wav）。欠けていれば設定画面の右上に項目名。受信モード・リプレイ・
  デモは対象外。既存の判定を読むだけで、条件は書き写さない
- 高温での充電の警告（v7・v7.1）: USB 接続中に MS5611 が 45°C を 30 秒超え続けたら
  地図に TOO HOT TO CHARGE と charge_hot.wav（60 秒ごと・最低音量 60）。電池の仕様は
  充電 0〜45°C。地図の段は電源異常と共用（異常 ＞ 高温 ＞ SW OFF）
- 電池低下のときの点滅（v7.1）: 電池低下の警告と同じ 3.5V でバックライトを 2 秒点灯・
  4 秒消灯。3.65V か USB で戻る（3.5V で戻すと入り切りをくり返す）。消灯中も本来の
  明るさは追い続ける（照度追従の立ち上がりで 2 秒の点灯が暗くならないように）
- 本体の回路図・PCB: 電池の逆接保護 Q4（AO3401A、D が電池側）＋ R52、PWR1 の
  ネットを VBAT_RAW に。C32 を 10µF 0805 に（10/20 に直したのが 0402 に戻っていた）。
  D5 を RB751S40（逆流が少ない。PCBA で実装）に。古いメモを整理
- IMU 基板の GND が IC1.16・C3 だけ分かれていたのをつないだ。J3 の値を 01x08 に。
  case_cover の部品番号を回路図と一致。GNSS 基板の裏面を GND ベタに（浮いていた
  19 個のビアがつながった）
- 音声 2 本（ready / charge_hot）は macOS の音声合成の仮音声
- docs: pons_power.md に Q4・P-ch FET 3 段の役割・電池の保護回路（DTP603048(PHR) の
  仕様書）・R39 を 2.2kΩ に戻さない理由（電池の最大充電 430mA も超える）・高温の警告・
  電池低下の点滅。README に GNSS の起動・本番前チェック・新しい警報・v7.1 の USB-C と
  充電時間、古い記述（v7 の実結線試験・無線の立ち上げ手順書の冒頭）を今の状態に。
  CLAUDE.md に BBR に書いた GNSS 設定が残る件と readiness.cpp
- kicad/.gitignore に *.pos

PONS_BOARD は V7 と V71 の両方でビルド OK（4,052,376 / 4,046,728 B）/
gen_wav_flash.py --check は 37 ファイル一致 / 本体 PCB の DRC は未配線 0・回路図と一致
（シルクの 6 件は意図どおり）/ IMU・カバー・GNSS 基板も未配線 0・回路図と一致 /
BOM の LCSC 番号は全 48 種類を JLC/LCSC の部品情報と照合 / 実機は未確認

Co-Authored-By: Claude Opus 5.5 <noreply@anthropic.com>
Parts:
- removed PWR1: 1s Lipo Power input, Connector_JST:JST_PH_S2B-PH-K_1x02_P2.00mm_Horizontal, symbol Connector:Conn_01x02_Pin
- added C5: 100u, Capacitor_SMD:C_1206_3216Metric, symbol Device:C
- SW1, SW2: FT Rotation Offset (none) -> 90
Connections:
- net +3V3: now also C5.1
- net GND: now also C5.2
Other:
- note removed: "BAT IN"
