File: kicad/IMU_murata/IMU_murata.kicad_sch (KiCad schematic)
At the start: 10 parts, among them IC1 SCH16T-K01-10, J1 Conn_01x08_Pin, J3 Conn_01x06_MountingPin

Commit message: 0.993 v7.1 基板の回路図と PCB を仕上げ、SW OFF のままの充電と電源異常を画面と音声で知らせるようにした
- power.cpp（新規）: USB の判定を usb_power_present() に一本化（v7.1 は VBUS を
  GPIO47 の ADC で測る）。電源経路の異常（2026-10-15 の充電 IC 焼損）を検出し、
  地図の POWER FAULT!! と power_fault.wav（30 秒ごと・最低音量 60）で知らせる。
  受信機は LINK_ST_PWR_FAULT を受けてトーン（同じ音声だとボートへの指示に聞こえる）
- v7.1: SW を OFF にしたまま USB で充電していると満充電にならない（Q3 のボディ
  ダイオード経由）。SW4 の OFF 側が GPIO40 を GND に落とすのを読み、地図に注意を出し
  1 度だけ読み上げる（charge_sw_off / charge_sw_on。排他グループ WAV_EXCL_CHARGE_SW）。
  移動中・ミラー中・リプレイ中・デモ中は出さない。判定に USB を入れない
  （VBUS が一瞬 4.3V を割ると 0V が本物の電池電圧として流れるため）。このあいだは
  電池低下の警告を止め、無線は RHAVE_VOLT を立てず LINK_ST_USB_SW_OFF、CSV は空欄
- 受信モードの電池表示を s55r42 の形に。SW OFF のまま USB の側は s5V / r5V
- backlight.cpp（新規）: v7.1 のバックライト PWM と VEML7700 の自動調光。
  飛行 CSV に lux / backlight 列
- E220 の M0/M1 は v7.1 で GPIO31 へ（GPIO47 は USB_SENS）
- 本体の回路図・PCB: SCH16T の J6 を逆順に（完成済みの FPC で J6-n ↔ J3-(9-n)）、
  F1 0805L035 → 0805L050（夏の充電で切れない）、R34/R35 を 10k/5.1k、C32 を 10µF 0805、
  SPI1 の SCK/MOSI/CS に 33Ω（R49〜R51）、スライドスイッチを MST-12D18G2 に、
  回路図とつながらない旧フットプリント（C33/R37/R38/R11 470Ω）を削除、DNP の BOM 除外、
  CUS-12TB の残骸とライブラリ登録を削除、メモの部品番号を v7.1 に
- GNSS 基板を 5 ピン（V_BCKUP）に。バックアップ電池は本体へ移した
- case_cover（照度センサー VEML7700）の kicad を追加。IMU ブレイクアウトの R2 を DNP
- 音声 3 本（power_fault / charge_sw_off / charge_sw_on）は macOS の音声合成の仮音声
- docs/pons_power.md（新規）。README の「自作の手順」を v7.1 に書き直し、
  SCH16T の配線の記述（J7・1:1 ケーブル）を J6・逆順に直した
- gen_wav_flash.py はコメント中の引用符付きの音声名も拾うので、録音前の名前を書かない

PONS_BOARD は V7 と V71 の両方でビルド OK（3,929,776 / 3,923,504 B）/
gen_wav_flash.py --check は 35 ファイル一致 / 本体 PCB の DRC は未配線 0・回路図と一致
（シルクの 6 件はボタンと USB の突起で意図どおり）/ GNSS 基板も未配線 0 / 実機は未確認

Co-Authored-By: Claude Opus 5.5 <noreply@anthropic.com>
Parts:
- R2: now not fitted
Changed lines of the file:
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@@
 		(on_board yes)
 		(in_pos_files yes)
-		(dnp no)
+		(dnp yes)
 		(fields_autoplaced yes)
 		(property "Reference" "R2"

Commit message: 0.994 GNSS の翌日起動を速くし、本番前チェック・高温充電の警告・電池低下の点滅を入れ、v7.1 基板の逆接保護と発注前の修正を仕上げた
- GNSS: AssistNow Autonomous を有効化（CFG-VALSET で RAM と BBR。settings.h の
  GNSS_USE_ANA。0 でも OFF を書き込む＝BBR に残った ON を消すため）。前日と同じ時間帯の
  起動が 23〜28 秒 → 3〜4 秒（BT1 が生きていること）。NAV-AOPSTATUS を 1Hz で受け、
  GNSS DETAIL 3 に ANA:ON data/use/calc、log.txt に「... after boot」（TTFF）・最初の
  測位の軌道の出どころ・10 分ごとの計算時間。ACK 待ちの間も imu_service_if_due() を
  呼ぶ（以前からの抜け）
- readiness.cpp（新規）: 本番前チェック。GNSS・IMU・ESKF・較正（マウント外れだけ。
  日付またぎは推測なので入れない＝台の上での APPLY を促さない）・地上の姿勢・設定画面の
  赤丸・USB・電池 50%・SD・無線（送信モード）がそろい、地上で止まっていたら 1 度だけ
  「準備完了」（ready.wav）。欠けていれば設定画面の右上に項目名。受信モード・リプレイ・
  デモは対象外。既存の判定を読むだけで、条件は書き写さない
- 高温での充電の警告（v7・v7.1）: USB 接続中に MS5611 が 45°C を 30 秒超え続けたら
  地図に TOO HOT TO CHARGE と charge_hot.wav（60 秒ごと・最低音量 60）。電池の仕様は
  充電 0〜45°C。地図の段は電源異常と共用（異常 ＞ 高温 ＞ SW OFF）
- 電池低下のときの点滅（v7.1）: 電池低下の警告と同じ 3.5V でバックライトを 2 秒点灯・
  4 秒消灯。3.65V か USB で戻る（3.5V で戻すと入り切りをくり返す）。消灯中も本来の
  明るさは追い続ける（照度追従の立ち上がりで 2 秒の点灯が暗くならないように）
- 本体の回路図・PCB: 電池の逆接保護 Q4（AO3401A、D が電池側）＋ R52、PWR1 の
  ネットを VBAT_RAW に。C32 を 10µF 0805 に（10/20 に直したのが 0402 に戻っていた）。
  D5 を RB751S40（逆流が少ない。PCBA で実装）に。古いメモを整理
- IMU 基板の GND が IC1.16・C3 だけ分かれていたのをつないだ。J3 の値を 01x08 に。
  case_cover の部品番号を回路図と一致。GNSS 基板の裏面を GND ベタに（浮いていた
  19 個のビアがつながった）
- 音声 2 本（ready / charge_hot）は macOS の音声合成の仮音声
- docs: pons_power.md に Q4・P-ch FET 3 段の役割・電池の保護回路（DTP603048(PHR) の
  仕様書）・R39 を 2.2kΩ に戻さない理由（電池の最大充電 430mA も超える）・高温の警告・
  電池低下の点滅。README に GNSS の起動・本番前チェック・新しい警報・v7.1 の USB-C と
  充電時間、古い記述（v7 の実結線試験・無線の立ち上げ手順書の冒頭）を今の状態に。
  CLAUDE.md に BBR に書いた GNSS 設定が残る件と readiness.cpp
- kicad/.gitignore に *.pos

PONS_BOARD は V7 と V71 の両方でビルド OK（4,052,376 / 4,046,728 B）/
gen_wav_flash.py --check は 37 ファイル一致 / 本体 PCB の DRC は未配線 0・回路図と一致
（シルクの 6 件は意図どおり）/ IMU・カバー・GNSS 基板も未配線 0・回路図と一致 /
BOM の LCSC 番号は全 48 種類を JLC/LCSC の部品情報と照合 / 実機は未確認

Co-Authored-By: Claude Opus 5.5 <noreply@anthropic.com>
Parts:
- J3: value Conn_01x06_MountingPin -> Conn_01x08_MountingPin
Changed lines of the file:
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@@
 			)
 		)
-		(property "Value" "Conn_01x06_MountingPin"
+		(property "Value" "Conn_01x08_MountingPin"
 			(at 228.6 83.8199 0)
 			(show_name no)
